File: rregatta.kicad_pcb (KiCad board)
At the start: 4 copper layers, 80 x 40 mm, 85 parts, among them J1 Program, J10 Horn, J2 Screw_Terminal_01x02, J3 Conn_01x02_Male, J4 5V out, J7 Light 2, J8 Light 1, J9 Light 3, Q1 HSBA3048, Q2 HSBA3048, Q3 HSBA3048, Q4 HSBA3048, SW1 Reset, U1 EUP3458, U2 AMS1117-3.3, U3 STM32F103C8T6, U4 SCT51240, U5 SCT51240, U6 SCT51240, U7 SCT51240, Y1 YSX531SL 8MHz, Y2 YST310S 32.768KHz

Commit message: update render
Parts:
- J10, J2, J7, J8, J9: footprint TerminalBlock:TerminalBlock_bornier-2_P5.08mm -> Custom:TerminalBlock_bornier-2_P5.08mm
