File: rregatta.kicad_sch (KiCad schematic)
At the start: 85 parts, among them J1 Program, J10 Horn, J2 Screw_Terminal_01x02, J3 Conn_01x02_Male, J4 5V out, J7 Light 2, J8 Light 1, J9 Light 3, Q1 HSBA3048, Q2 HSBA3048, Q3 HSBA3048, Q4 HSBA3048, SW1 Reset, U1 EUP3458, U2 AMS1117-3.3, U3 STM32F103C8T6, U4 SCT51240, U5 SCT51240, U6 SCT51240, U7 SCT51240, Y1 YSX531SL 8MHz, Y2 YST310S 32.768KHz

Commit message: update render
Parts:
- J10, J2, J7, J8, J9: footprint TerminalBlock:TerminalBlock_bornier-2_P5.08mm -> Custom:TerminalBlock_bornier-2_P5.08mm
Changed lines of the file:
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@@
       (effects (font (size 1.27 1.27)) (justify left))
     )
-    (property "Footprint" "TerminalBlock:TerminalBlock_bornier-2_P5.08mm" (id 2) (at 267.081 29.972 0)
+    (property "Footprint" "Custom:TerminalBlock_bornier-2_P5.08mm" (id 2) (at 267.081 29.972 0)
       (effects (font (size 1.27 1.27)) hide)
     )
@@
       (effects (font (size 1.27 1.27)) (justify left))
     )
-    (property "Footprint" "TerminalBlock:TerminalBlock_bornier-2_P5.08mm" (id 2) (at 265.43 137.414 0)
+    (property "Footprint" "Custom:TerminalBlock_bornier-2_P5.08mm" (id 2) (at 265.43 137.414 0)
       (effects (font (size 1.27 1.27)) hide)
     )
@@
       (effects (font (size 1.27 1.27)) (justify left))
     )
-    (property "Footprint" "TerminalBlock:TerminalBlock_bornier-2_P5.08mm" (id 2) (at 269.748 61.341 0)
+    (property "Footprint" "Custom:TerminalBlock_bornier-2_P5.08mm" (id 2) (at 269.748 61.341 0)
       (effects (font (size 1.27 1.27)) hide)
     )
@@
       (effects (font (size 1.27 1.27)) (justify left))
     )
-    (property "Footprint" "TerminalBlock:TerminalBlock_bornier-2_P5.08mm" (id 2) (at 268.732 91.44 0)
+    (property "Footprint" "Custom:TerminalBlock_bornier-2_P5.08mm" (id 2) (at 268.732 91.44 0)
       (effects (font (size 1.27 1.27)) hide)
     )
@@
     (property "Reference" "J2" (id 0) (at 42.164 38.1168 0))
     (property "Value" "Screw_Terminal_01x02" (id 1) (at 42.164 35.5799 0))
-    (property "Footprint" "TerminalBlock:TerminalBlock_bornier-2_P5.08mm" (id 2) (at 42.164 30.607 0)
+    (property "Footprint" "Custom:TerminalBlock_bornier-2_P5.08mm" (id 2) (at 42.164 30.607 0)
       (effects (font (size 1.27 1.27)) hide)
     )
@@
     )
     (path "/bb60f894-002b-469c-bb5c-0f0d44c12cb4"
-      (reference "J2") (unit 1) (value "Screw_Terminal_01x02") (footprint "TerminalBlock:TerminalBlock_bornier-2_P5.08mm")
+      (reference "J2") (unit 1) (value "Screw_Terminal_01x02") (footprint "Custom:TerminalBlock_bornier-2_P5.08mm")
     )
     (path "/6f913f83-e3b1-43e5-a237-71342f04d8ca"
@@
     )
     (path "/3c1e0dd8-c37f-4efa-bf6b-7ef4e337d7b6"
-      (reference "J7") (unit 1) (value "Light 2") (footprint "TerminalBlock:TerminalBlock_bornier-2_P5.08mm")
+      (reference "J7") (unit 1) (value "Light 2") (footprint "Custom:TerminalBlock_bornier-2_P5.08mm")
     )
     (path "/9e61dd8a-a378-457a-a1a4-32d2c882a353"
-      (reference "J8") (unit 1) (value "Light 1") (footprint "TerminalBlock:TerminalBlock_bornier-2_P5.08mm")
+      (reference "J8") (unit 1) (value "Light 1") (footprint "Custom:TerminalBlock_bornier-2_P5.08mm")
     )
     (path "/ae3e599c-9366-488d-8bd4-2e3fac3f8d9a"
-      (reference "J9") (unit 1) (value "Light 3") (footprint "TerminalBlock:TerminalBlock_bornier-2_P5.08mm")
+      (reference "J9") (unit 1) (value "Light 3") (footprint "Custom:TerminalBlock_bornier-2_P5.08mm")
     )
     (path "/41a92c8f-6103-4f7a-a1e4-3873b0276002"
-      (reference "J10") (unit 1) (value "Horn") (footprint "TerminalBlock:TerminalBlock_bornier-2_P5.08mm")
+      (reference "J10") (unit 1) (value "Horn") (footprint "Custom:TerminalBlock_bornier-2_P5.08mm")
     )
     (path "/a812acfe-de29-4d43-9292-15e24f4fac35"
